Commit message: Fix: Correct robot model asymmetry in XML and update policies
- Symmetrized joint limits, axes, and collision geometry in the MJCF (robot.xml) to fix balance issues.
- Updated and cleaned up policy files, removing outdated models.
- Adjusted reward function parameters in the training configuration.
- Deleted obsolete posture fixing script.

File: pointfootGym/resources/robots/pointfoot/PF_TRON1A/urdf/robot.urdf (robot description, URDF)
Before this commit: robot point_foot, 12 links, 11 joints
Joints:
- joint knee_L_Joint: limit lower=-0.872665 upper=1.396263 effort=80 velocity=20 -> lower=-0.872665 upper=1.396263 effort=80 velocity=50
