Commit message: Complete refactor of pointfootGym and pointfootMujoco projects
- Restructured pointfootGym environment configuration and training scripts
- Updated pointfootMujoco controller and policy system
- Synchronized robot model parameters across both projects
- Removed legacy controller files and simplified architecture
- Added new gitattributes configuration

🤖 Generated with [Claude Code](https://claude.ai/code)

Co-Authored-By: Claude <noreply@anthropic.com>

File: pointfootGym/resources/robots/pointfoot/PF_TRON1A/urdf/robot.urdf (robot description, URDF)
Before this commit: robot point_foot, 12 links, 11 joints
Joints:
- joint abad_R_Joint: limit lower=-0.38397 upper=1.39626 effort=80.0 velocity=20.0 -> lower=-1.39626 upper=0.38397 effort=80.0 velocity=20.0

Commit message: Update robot model URDF and XML files
- Update base_Link center of mass position in URDF
- Adjust joint limits and inertial properties in both URDF and XML
- Synchronize collision geometry and mesh references
- Fine-tune joint velocity limits for knee joint

🤖 Generated with [Claude Code](https://claude.ai/code)

Co-Authored-By: Claude <noreply@anthropic.com>

File: pointfootGym/resources/robots/pointfoot/PF_TRON1A/urdf/robot.urdf (robot description, URDF)
Before this commit: robot point_foot, 12 links, 11 joints
Joints:
- joint knee_L_Joint: limit lower=-0.872665 upper=1.396263 effort=80 velocity=50 -> lower=-0.872665 upper=1.396263 effort=80 velocity=20
